Commit message: adding gripper !!!

File: QARM/urdf/QARM_new.urdf (robot description, URDF)
Before this commit: robot QARM, 6 links, 5 joints
Links:
- removed link END_EFFECTOR
- added link END_EFFECTOR_BASE, mass 0.257; collision mesh filename=package://QARM/meshes/END_EFFECTOR_BASE.STL; visual mesh filename=package://QARM/meshes/END_EFFECTOR_BASE.STL
- added link LINK1A, mass 0.075987; collision mesh filename=package://QARM/meshes/LINK1A.STL; visual mesh filename=package://QARM/meshes/LINK1A.STL
- added link LINK1B, mass 0; collision mesh filename=package://QARM/meshes/LINK1B.STL; visual mesh filename=package://QARM/meshes/LINK1B.STL
- added link LINK2A, mass 0.0291073155718739; collision mesh filename=package://QARM/meshes/LINK2A.STL; visual mesh filename=package://QARM/meshes/LINK2A.STL
- added link LINK2B, mass 0.0291073142953973; collision mesh filename=package://QARM/meshes/LINK2B.STL; visual mesh filename=package://QARM/meshes/LINK2B.STL
Joints:
- added joint JOINT1A: type revolute, parent END_EFFECTOR_BASE, child LINK1A, origin xyz=0.03075 0.0345 0.016987 rpy=0 1.5708 0, axis 0 0 1, limit lower=0 upper=0 effort=0 velocity=0
- added joint JOINT1B: type revolute, parent END_EFFECTOR_BASE, child LINK1B, origin xyz=0.03075 0.0345 0.016987 rpy=0 0 -0.58368, axis 0 0 1, limit lower=0 upper=0 effort=0 velocity=0
- added joint JOINT2A: type revolute, parent LINK1A, child LINK2A, origin xyz=0 0.07 0 rpy=0 0 -0.094813, axis 0 0 1, limit lower=0 upper=0 effort=0 velocity=0
- added joint JOINT2B: type revolute, parent LINK1B, child LINK2B, origin xyz=0 0.07 0 rpy=0 0 0.055781, axis 0 0 -1, limit lower=0 upper=0 effort=0 velocity=0
- joint WRIST: child END_EFFECTOR -> END_EFFECTOR_BASE
