Commit message: cleaning genesis tests and creating base simulation script (udp for real and no udp for rl)

File: genesis/QARM/urdf/QARM.urdf (robot description, URDF)
Before this commit: robot QARM, 6 links, 5 joints
Links:
- removed link END-EFFECTOR
- added link END_EFFECTOR_BASE, mass 0.257; collision mesh filename=../meshes/END_EFFECTOR_BASE.STL; visual mesh filename=../meshes/END_EFFECTOR_BASE.STL
- link BICEP: mass 0.706073338310231 -> 0.4591; geometry collision mesh filename=../meshes/BICEP.STL; visual mesh filename=../meshes/BICEP.STL
- link FOREARM: mass 0.4296669212638 -> 0.269; geometry collision mesh filename=../meshes/FOREARM.STL; visual mesh filename=../meshes/FOREARM.STL
- link YAW: mass 0.701518504018672 -> 0.7906; geometry collision mesh filename=../meshes/YAW.STL; visual mesh filename=../meshes/YAW.STL
- link base_link: geometry collision mesh filename=../meshes/base_link.STL; visual mesh filename=../meshes/base_link.STL
Joints:
- joint ELBOW: limit lower=-1.658 upper=1.309 effort=0 velocity=0 -> lower=-1.658 upper=1.309 effort=100.0 velocity=1.57; origin xyz=0.0500000000000004 -0.350000000000015 0 rpy=0 0 -1.42889927219074 -> xyz=0.0500 -0.3500 0 rpy=0 0 -1.42889927219074
- joint SHOULDER: limit lower=-1.483 upper=1.483 effort=0 velocity=0 -> lower=-1.483 upper=1.483 effort=100.0 velocity=1.57; origin xyz=0 0 0.1397714 rpy=-1.5707963267949 0 0 -> xyz=0 0 0.1400 rpy=-1.5707963267949 0 0
- joint WRIST: child END-EFFECTOR -> END_EFFECTOR_BASE; limit lower=-3.010 upper=3.010 effort=0 velocity=0 -> lower=-2.792 upper=2.792 effort=100.0 velocity=1.57; origin xyz=0.0336611536380097 0.235607569369425 0 rpy=-1.5707963267949 0 -0.141897054604159 -> xyz=0.03535533905932738 0.24748737341529164 0.0 rpy=-1.5707963267949 0 -0.141897054604159
- joint YAW: limit lower=-2.967 upper=2.967 effort=0 velocity=0 -> lower=-2.967 upper=2.967 effort=100.0 velocity=1.57

Commit message: visualization of quintics coeffs

File: genesis/QARM/urdf/QARM.urdf (robot description, URDF)
Before this commit: robot QARM, 6 links, 5 joints
Links:
- link END_EFFECTOR_BASE: geometry collision box size=0.02 0.10 0.15; visual box size=0.02 0.10 0.15
