Commit message: Testing camera sensor

File: genesis/QARM/urdf/QARM.urdf (robot description, URDF)
Before this commit: robot QARM, 6 links, 5 joints
Links:
- removed link END_EFFECTOR_BASE
- added link END_EFFECTOR, mass 0.257; collision box size=0.02 0.10 0.15; visual box size=0.02 0.10 0.15
Joints:
- joint WRIST: child END_EFFECTOR_BASE -> END_EFFECTOR

File: genesis/QARM/urdf/gripper.urdf (robot description, URDF)
Before this commit: robot qarm_gripper, 5 links, 4 joints
Links:
- link END_EFFECTOR_BASE: geometry collision mesh filename=package://QARM/meshes/END_EFFECTOR.STL; visual mesh filename=package://QARM/meshes/test.stl

File: genesis/QARM/urdf/qarm_with_gripper.urdf (robot description, URDF)
Before this commit: robot QARM, 11 links, 10 joints
Links:
- removed link END-EFFECTOR
- removed link Link1A
- removed link Link1B
- removed link Link2A
- removed link Link2B
- removed link gripper_base_link
- added link END_EFFECTOR, mass 0.025331269641348; collision mesh filename=../meshes/END_EFFECTOR.stl; visual mesh filename=../meshes/END_EFFECTOR.stl
- added link END_EFFECTOR_BASE, mass 0.32859; collision mesh filename=../meshes/END_EFFECTOR_BASE.stl; visual mesh filename=../meshes/END_EFFECTOR_BASE.stl
- added link LINK1A, mass 0.075987; collision mesh filename=../meshes/LINK1A.stl; visual mesh filename=../meshes/LINK1A.stl
- added link LINK1B, mass 0.075987; collision mesh filename=../meshes/LINK1B.stl; visual mesh filename=../meshes/LINK1B.stl
- added link LINK2A, mass 0.0291073155718739; collision mesh filename=../meshes/LINK2A.stl; visual mesh filename=../meshes/LINK2A.stl
- added link LINK2B, mass 0.0291073155718739; collision mesh filename=../meshes/LINK2B.stl; visual mesh filename=../meshes/LINK2B.stl
- link BICEP: geometry collision mesh filename=../meshes/BICEP.stl; visual mesh filename=../meshes/BICEP.stl
- link FOREARM: geometry collision mesh filename=../meshes/FOREARM.stl; visual mesh filename=../meshes/FOREARM.stl
- link YAW: geometry collision mesh filename=../meshes/YAW.stl; visual mesh filename=../meshes/YAW.stl
- link base_link: geometry collision mesh filename=../meshes/base_link.stl; visual mesh filename=../meshes/base_link.stl
Joints:
- removed joint Joint1A
- removed joint Joint1B
- removed joint Joint2A
- removed joint Joint2B
- removed joint gripper_mount
- added joint GRIPPER_MOUNT: type fixed, parent END_EFFECTOR, child END_EFFECTOR_BASE, origin xyz=0 0 0 rpy=0 0 0
- added joint JOINT1A: type revolute, parent END_EFFECTOR_BASE, child LINK1A, origin xyz=0.01 0.03075 0.0399 rpy=0 0 0, axis 1 0 0, limit lower=-0.9 upper=0.9 effort=10 velocity=5
- added joint JOINT1B: type revolute, parent END_EFFECTOR_BASE, child LINK1B, origin xyz=0.01 -0.03075 0.0399 rpy=0 0 0, axis 1 0 0, limit lower=-0.9 upper=0.9 effort=10 velocity=5
- added joint JOINT2A: type revolute, parent LINK1A, child LINK2A, origin xyz=-0.000842 -0.000324 0.07 rpy=0 0 0, axis 1 0 0, limit lower=-0.9 upper=0.9 effort=10 velocity=5
- added joint JOINT2B: type revolute, parent LINK1B, child LINK2B, origin xyz=-0.000842 0.000324 0.07 rpy=0 0 0, axis 1 0 0, limit lower=-0.9 upper=0.9 effort=10 velocity=5
- joint WRIST: child END-EFFECTOR -> END_EFFECTOR
